Commit message: 20210623

File: magician_description/urdf/magician.urdf.orig.xacro (robot description, xacro)
@@ -9,7 +9,7 @@
   <xacro:property name="joint1_lower" value="-2.1816"/>
   <xacro:property name="joint1_upper" value="2.1816"/>
-  <xacro:property name="joint2_lower" value="-0.35"/>
+  <xacro:property name="joint2_lower" value="0.35"/>
   <xacro:property name="joint2_upper" value="1.57"/>
-  <xacro:property name="joint3_lower" value="-0.62"/>
+  <xacro:property name="joint3_lower" value="0.62"/>
   <xacro:property name="joint3_upper" value="1.57"/>
   <link name="world"/>

Commit message: 20210627

File: magician_description/urdf/magician.urdf.orig.xacro (robot description, xacro)
@@ -616,5 +616,5 @@
       xyz="0 0 0" />
   </joint>
-  <link name="magician_end_effctor"/>
+  <link name="magician_end_effector"/>
   <joint
     name="magician_end_link_joint1"
@@ -626,5 +626,5 @@
       link="magician_end_link" />
     <child
-      link="magician_end_effctor" />
+      link="magician_end_effector" />
     <axis
       xyz="0 0 0" />

File: magician_description/urdf/magician.urdf.xacro (robot description, xacro)
@@ -616,5 +616,5 @@
       xyz="0 0 0" />
   </joint>
-  <link name="magician_end_effctor"/>
+  <link name="magician_end_effector"/>
   <joint
     name="magician_end_link_joint1"
@@ -626,5 +626,5 @@
       link="magician_end_link" />
     <child
-      link="magician_end_effctor" />
+      link="magician_end_effector" />
     <axis
       xyz="0 0 0" />

File: magician_description/urdf/magician_ikfast.urdf (robot description, URDF)
Before this commit: robot magician, 13 links, 12 joints
Links:
- removed link magician_end_effctor
- added link magician_end_effector
Joints:
- joint magician_end_link_joint1: child magician_end_effctor -> magician_end_effector

File: magician_description/urdf/magician_open_chain.urdf.xacro (robot description, xacro)
@@ -575,5 +575,5 @@
       xyz="0 0 0" />
   </joint>
-  <link name="magician_end_effctor"/>
+  <link name="magician_end_effector"/>
   <joint
     name="magician_end_link_joint1"
@@ -585,5 +585,5 @@
       link="magician_end_link" />
     <child
-      link="magician_end_effctor" />
+      link="magician_end_effector" />
     <axis
       xyz="0 0 0" />
