Commit message: 20210629

File: magician_description/urdf/magician.urdf.xacro (robot description, xacro)
@@ -7,4 +7,5 @@
   <xacro:include filename="$(find magician_description)/urdf/magician.gazebo" />
   <xacro:include filename="$(find magician_description)/urdf/magician_transmission.xacro" />
+<!--
   <xacro:property name="joint1_lower" value="-2.1816"/>
   <xacro:property name="joint1_upper" value="2.1816"/>
@@ -13,4 +14,15 @@
   <xacro:property name="joint3_lower" value="-0.62"/>
   <xacro:property name="joint3_upper" value="1.57"/>
+-->
+  <xacro:property name="joint1_lower" value="-1.57"/>
+  <xacro:property name="joint1_upper" value="1.57"/>
+  <xacro:property name="joint2_lower" value="0"/>
+  <xacro:property name="joint2_upper" value="1.48"/>
+  <xacro:property name="joint3_lower" value="-1.17"/>
+  <xacro:property name="joint3_upper" value="1.57"/>
+  <xacro:property name="joint_velocity" value="0.5"/> <!-- mm/s   ???? -->
+<!--
+  <xacro:property name="joint_velocity" value="1.57"/>
+-->
   <link name="world"/>
   <link name="magician_origin"/>
@@ -137,5 +149,5 @@
       upper="${joint1_upper}"
       effort="6"
-      velocity="1.57" />
+      velocity="${joint_velocity}" />
   </joint>
   <link
@@ -195,5 +207,5 @@
       upper="${joint2_upper}"
       effort="6"
-      velocity="1.57" />
+      velocity="${joint_velocity}" />
   </joint>
   <link
@@ -253,5 +265,5 @@
       upper="${-1*joint2_lower}"
       effort="6"
-      velocity="1.57" />
+      velocity="${joint_velocity}" />
     <mimic
       joint="magician_joint2"
@@ -291,5 +303,5 @@
       upper="${joint3_upper}"
       effort="6"
-      velocity="1.57" />
+      velocity="${joint_velocity}" />
   </joint>
   <link
@@ -349,5 +361,5 @@
       upper="${-1*joint3_lower}"
       effort="6"
-      velocity="1.57" />
+      velocity="${joint_velocity}" />
     <mimic
       joint="magician_joint3"
@@ -596,5 +608,5 @@
       upper="${-1*joint1_lower}"
       effort="6"
-      velocity="1.57" />
+      velocity="${joint_velocity}" />
     <mimic
       joint="magician_joint1"

Commit message: 20210207

File: magician_description/urdf/magician.urdf.xacro (robot description, xacro)
@@ -21,8 +21,5 @@
   <xacro:property name="joint3_lower" value="-1.17"/>
   <xacro:property name="joint3_upper" value="1.57"/>
-  <xacro:property name="joint_velocity" value="0.5"/> <!-- mm/s   ???? -->
-<!--
-  <xacro:property name="joint_velocity" value="1.57"/>
--->
+  <xacro:property name="joint_velocity" value="1.57"/> <!-- rad/s   ???? -->
   <link name="world"/>
   <link name="magician_origin"/>

Commit message: 20210705

File: magician_description/urdf/magician.urdf.xacro (robot description, xacro)
@@ -7,5 +7,4 @@
   <xacro:include filename="$(find magician_description)/urdf/magician.gazebo" />
   <xacro:include filename="$(find magician_description)/urdf/magician_transmission.xacro" />
-<!--
   <xacro:property name="joint1_lower" value="-2.1816"/>
   <xacro:property name="joint1_upper" value="2.1816"/>
@@ -14,5 +13,5 @@
   <xacro:property name="joint3_lower" value="-0.62"/>
   <xacro:property name="joint3_upper" value="1.57"/>
--->
+<!--
   <xacro:property name="joint1_lower" value="-1.57"/>
   <xacro:property name="joint1_upper" value="1.57"/>
@@ -21,7 +20,10 @@
   <xacro:property name="joint3_lower" value="-1.17"/>
   <xacro:property name="joint3_upper" value="1.57"/>
+-->
   <xacro:property name="joint_velocity" value="1.57"/> <!-- rad/s   ???? -->
   <link name="world"/>
+<!--
   <link name="magician_origin"/>
+-->
   <joint
     name="world_joint"
@@ -33,5 +35,5 @@
       link="world" />
     <child
-      link="magician_origin" />
+      link="magician_base" />
     <axis
       xyz="0 0 0" />
@@ -77,4 +79,5 @@
     </collision>
   </link>
+<!--
   <joint
     name="magician_origin_joint1"
@@ -90,4 +93,5 @@
       xyz="0 0 0" />
   </joint>
+-->
   <link
     name="magician_link1">
@@ -639,3 +643,15 @@
       xyz="0 0 0" />
   </joint>
+  <link name="magician_tool0"/>
+  <joint
+    name="magician_tool0_joint"
+    type="fixed">
+    <origin
+      xyz="0.041 0.0 0.0"
+      rpy="3.1415926535897932 0 0" />
+    <parent
+      link="magician_end_effector" />
+    <child
+      link="magician_tool0" />
+  </joint>
 </robot>

Commit message: 20210713

File: magician_description/urdf/magician.urdf.xacro (robot description, xacro)
@@ -649,7 +649,7 @@
     <origin
       xyz="0.041 0.0 0.0"
-      rpy="3.1415926535897932 0 0" />
-    <parent
-      link="magician_end_effector" />
+      rpy="0 0 0" />
+    <parent
+      link="magician_arm_end" />
     <child
       link="magician_tool0" />
